Commit message: updated tag names

File: models/tag_box2.urdf.xacro (robot description, xacro)
@@ -12,7 +12,7 @@
       <geometry>
         <!--AR Track Alvar. -->
-        <mesh filename="package://tag_world/meshes/tags$(arg tag_num).dae" />
+        <!--<mesh filename="package://tag_world/meshes/tags$(arg tag_num).dae" />-->
         <!-- April Tags. -->
-        <!-- <mesh filename="package://tag_world/meshes/apriltags$(arg tag_num).dae" /> -->
+        <mesh filename="package://tag_world/meshes/apriltags$(arg tag_num).dae" />
       </geometry>
     </visual>
