Commit message: cleaned up documentation

File: models/tag_box.urdf.xacro (robot description, xacro)
@@ -1,26 +1,22 @@
 <?xml version="1.0"?>
-<!-- This is for loading a single tag as a flat box. -->
-<robot name="tag_box">
+<robot name="tag_box" xmlns:xacro="http://www.ros.org/wiki/xacro">
   <link name="tag_link">
     <inertial>
-      <origin xyz="0 0 0" />
-      <mass value="0.001" />
+      <origin xyz="0 0 0.15" />
+      <mass value="0.3" />
       <inertia  ixx="1.0" ixy="0.0"  ixz="0.0"  iyy="1.0"  iyz="0.0"  izz="1.0" />
     </inertial>
     <visual>
-      <origin xyz="0 0 0"/>
+      <origin xyz="0 0 0.15"/>
       <geometry>
-        <mesh filename="package://tag_world/meshes/tag$(arg tag_num).dae" />
+        <mesh filename="package://tag_world/meshes/tags$(arg tag_num).dae" />
       </geometry>
     </visual>
     <collision>
-      <origin xyz="0 0 0"/>
+      <origin xyz="0 0 0.15"/>
       <geometry>
-        <box size="0.1 0.1 0.001" />
+        <box size="0.3 0.3 0.3" />
       </geometry>
     </collision>
   </link>
-  <!--<gazebo reference="base_link">
-    <material>Gazebo/Blue</material>
-  </gazebo>-->
 </robot>

File: models/tag_box2.urdf.xacro (robot description, xacro)
@@ -82,41 +82,4 @@
     <origin xyz="0 0 0" rpy="3.1416 0 1.571"/>
   </joint>
-  <!--
-  <link name="ar_marker_${$(arg tag_num)*6}"></link>
-  <joint name="ar_marker_${$(arg tag_num)*6}_joint" type="fixed">
-    <parent link="tag_link" />
-    <child link="ar_marker_${$(arg tag_num)*6}" />
-    <origin xyz="0.15 0 0.15" rpy="1.571 0 1.571"/>
-  </joint>
-  <link name="ar_marker_${$(arg tag_num)*6+1}"></link>
-  <joint name="ar_marker_${$(arg tag_num)*6+1}_joint" type="fixed">
-    <parent link="tag_link" />
-    <child link="ar_marker_${$(arg tag_num)*6+1}" />
-    <origin xyz="0 -0.15 0.15" rpy="1.571 0 0"/>
-  </joint>
-  <link name="ar_marker_${$(arg tag_num)*6+2}"></link>
-  <joint name="ar_marker_${$(arg tag_num)*6+2}_joint" type="fixed">
-    <parent link="tag_link" />
-    <child link="ar_marker_${$(arg tag_num)*6+2}" />
-    <origin xyz="-0.15 0 0.15" rpy="-1.571 0 1.571"/>
-  </joint>
-  <link name="ar_marker_${$(arg tag_num)*6+3}"></link>
-  <joint name="ar_marker_${$(arg tag_num)*6+3}_joint" type="fixed">
-    <parent link="tag_link" />
-    <child link="ar_marker_${$(arg tag_num)*6+3}" />
-    <origin xyz="0 0.15 0.15" rpy="-1.571 0 0"/>
-  </joint>
-  <link name="ar_marker_${$(arg tag_num)*6+4}"></link>
-  <joint name="ar_marker_${$(arg tag_num)*6+4}_joint" type="fixed">
-    <parent link="tag_link" />
-    <child link="ar_marker_${$(arg tag_num)*6+4}" />
-    <origin xyz="0 0 0.3" rpy="0 0 0"/>
-  </joint>
-  <link name="ar_marker_${$(arg tag_num)*6+5}"></link>
-  <joint name="ar_marker_${$(arg tag_num)*6+5}_joint" type="fixed">
-    <parent link="tag_link" />
-    <child link="ar_marker_${$(arg tag_num)*6+5}" />
-    <origin xyz="0 0 0" rpy="3.1416 0 1.571"/>
-  </joint>-->
   <gazebo reference="base_link">
     <turnGravityOff>false</turnGravityOff>

Commit message: adding pole

File: models/tag_box.urdf.xacro (robot description, xacro)
@@ -10,5 +10,5 @@
       <origin xyz="0 0 0.15"/>
       <geometry>
-        <mesh filename="package://tag_world/meshes/tags$(arg tag_num).dae" />
+        <mesh filename="package://tag_world/meshes/apriltags$(arg tag_num).dae" />
       </geometry>
     </visual>

File: models/tag_box3.urdf.xacro (robot description, xacro)
@@ -1,5 +1,42 @@
 <?xml version="1.0"?>
-<!-- This is for loading a box with different tags on each side. -->
+<!-- This is for loading a box with different tags on each side. Adds a pole. -->
 <robot name="box" xmlns:xacro="http://www.ros.org/wiki/xacro">
+  <xacro:property name="pole_height" value="0.4" />
+  <xacro:property name="pole_radius" value="0.05" />
+  <xacro:property name="box_width"   value="0.2" />
+  <material name="light_grey"><color rgba="0.4 0.4 0.4 1.0" /></material>
+  <link name="base_link"></link>
+  <joint name="pole_joint" type="fixed">
+    <parent link="base_link" />
+    <child link="pole_link" />
+    <origin xyz="0 0 0" rpy="0 0 0" />
+    <axis xyz="0 0 0" />
+  </joint>
+  <link name="pole_link">
+    <inertial>
+      <origin xyz="0 0 ${pole_height/2}" />
+      <mass value="10.0" />
+      <inertia  ixx="0.4" ixy="0.0"  ixz="0.0"  iyy="0.4"  iyz="0.0"  izz="0.2" />
+    </inertial>
+    <visual>
+      <origin xyz="0 0 ${pole_height/2}"/>
+      <geometry>
+        <cylinder length="${pole_height}" radius="${pole_radius}"/>
+      </geometry>
+      <material name="light_grey"/>
+    </visual>
+    <collision>
+      <origin xyz="0 0 ${pole_height/2}"/>
+      <geometry>
+        <cylinder length="${pole_height}" radius="${pole_radius}"/>
+      </geometry>
+    </collision>
+  </link>
+  <joint name="ar_tag_joint" type="fixed">
+    <parent link="pole_link" />
+    <child link="tag_link" />
+    <origin xyz="0 0 ${pole_height}" rpy="0 0 0" />
+    <axis xyz="0 1 0" />
+  </joint>
   <link name="tag_link">
     <inertial>
@@ -9,5 +46,5 @@
     </inertial>
     <visual>
-      <origin xyz="0 0 0.15"/>
+      <origin xyz="0 0 ${box_width/2}"/>
       <geometry>
         <!--AR Track Alvar. -->
@@ -18,17 +55,10 @@
     </visual>
     <collision>
-      <origin xyz="0 0 0.15"/>
+      <origin xyz="0 0 ${box_width/2}"/>
       <geometry>
-        <box size="0.3 0.3 0.3" />
+        <box size="${box_width} ${box_width} ${box_width}" />
       </geometry>
     </collision>
   </link>
-  <link name="base_link"></link>
-  <joint name="ar_tag_joint" type="fixed">
-    <parent link="base_link" />
-    <child link="tag_link" />
-    <origin xyz="0 0 0.19" rpy="0 0 0" />
-    <axis xyz="0 1 0" />
-  </joint>
   <!-- Robot 0 has tags 0 to 5, robot 1 has tags 6 to 10 etc.
        From the perspective of the host robot, the order is:
@@ -46,5 +76,5 @@
        -->
   <xacro:property name="num" value="$(arg tag_num)" />
-  <xacro:property name="width" value="0.3"/>
+  <xacro:property name="width" value="${box_width}"/>
   <link name="ar_marker_${num*6}"></link>
   <joint name="ar_marker_${num*6}_joint" type="fixed">

Commit message: changing meshes to match multi_jackal

File: models/tag_box.urdf.xacro (robot description, xacro)
@@ -10,5 +10,5 @@
       <origin xyz="0 0 0.15"/>
       <geometry>
-        <mesh filename="package://tag_world/meshes/apriltags$(arg tag_num).dae" />
+        <mesh filename="package://tag_world/meshes/apriltags/apriltags$(arg tag_num).dae" />
       </geometry>
     </visual>

File: models/tag_box2.urdf.xacro (robot description, xacro)
@@ -12,7 +12,7 @@
       <geometry>
         <!--AR Track Alvar. -->
-        <!--<mesh filename="package://tag_world/meshes/tags$(arg tag_num).dae" />-->
+        <!--<mesh filename="package://tag_world/meshes/alvartags/alvartags$(arg tag_num).dae" />-->
         <!-- April Tags. -->
-        <mesh filename="package://tag_world/meshes/apriltags$(arg tag_num).dae" />
+        <mesh filename="package://tag_world/meshes/apriltags/apriltags$(arg tag_num).dae" />
       </geometry>
     </visual>

File: models/tag_box3.urdf.xacro (robot description, xacro)
@@ -49,7 +49,7 @@
       <geometry>
         <!--AR Track Alvar. -->
-        <!--<mesh filename="package://tag_world/meshes/tags$(arg tag_num).dae" />-->
+        <!--<mesh filename="package://tag_world/meshes/alvartags/alvartags$(arg tag_num).dae" />-->
         <!-- April Tags. -->
-        <mesh filename="package://tag_world/meshes/apriltags$(arg tag_num).dae" />
+        <mesh filename="package://tag_world/meshes/apriltags/apriltags$(arg tag_num).dae" />
       </geometry>
     </visual>
